Commit message: 3d

File: arm_3.urdf (robot description, URDF)
Before this commit: robot three_dof_arm, 4 links, 3 joints
Links:
- link link1: geometry collision cylinder length=1.50 radius=0.04; visual cylinder length=1.50 radius=0.04
- link link2: geometry collision cylinder length=1.50 radius=0.04; visual cylinder length=1.50 radius=0.04
- link link3: geometry collision cylinder length=1.20 radius=0.04; visual cylinder length=1.20 radius=0.04
Joints:
- joint joint2: origin xyz=0 0 0.50 rpy=0 0 0 -> xyz=0 0 1.50 rpy=0 0 0
- joint joint3: origin xyz=0 0 0.50 rpy=0 0 0 -> xyz=0 0 1.50 rpy=0 0 0
